Commit message: Mount the IMU frame and give the camera a nominal lens model
- Rotate imu_mount -90 degrees about z, matching the chip's x right and y forward found by tilting Gerry
- Load a nominal OV5647 camera_info from config/ov5647.yaml so Foxglove can project the image
- Publish camera frames best effort so Wi-Fi loss drops a frame instead of stalling
- Note pack0 reading high under servo load, and archive what Gerry confirmed

File: src/hexapod/urdf/hexapod.urdf.xacro (robot description, xacro)
@@ -164,8 +164,8 @@
     </joint>
     <link name="ultrasonic"/>
-    <joint name="imu_mount" type="fixed">  <!-- axes unchecked -->
+    <joint name="imu_mount" type="fixed">  <!-- the chip's x points right, its y forward -->
         <parent link="base_link"/>
         <child link="imu"/>
-        <origin xyz="0.0399 -0.0086 0.0375"/>
+        <origin xyz="0.0399 -0.0086 0.0375" rpy="0 0 ${-pi/2}"/>
     </joint>
     <link name="imu"/>
